File: KiCad_PCB/Riscduino_Debug_Rev1.1/Riscduino_Debug.kicad_pcb (KiCad board)
At the start: 2 copper layers, 70.6 x 53.7 mm, 86 parts, among them J1 Conn_01x06_Pin, J10 USB_B_Micro, J11 Conn_01x10_Pin, J2 Conn_01x08_Pin, J3 Conn_01x01, J4 Conn_02x04_Odd_Even, J5 ISP, J6 Conn_01x01, J7 Conn_01x01, J8 Conn_01x01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

Commit message: Update
Parts:
- removed TP1: TestPoint, Connector_PinHeader_2.54mm:PinHeader_1x01_P2.54mm_Vertical
- added R33: R, Resistor_SMD:R_0603_1608Metric_Pad0.98x0.95mm_HandSolder, F.Cu at (137.2, 99.3)
Connections:
- J2 pad 5: +1V8 -> +5V
Routing:
- net USER_FLASH_IO2: track 60.1 -> 154.1 mm
- net GND: track 377.2 -> 448.8 mm, vias 11 -> 6
- net CARAVEL_FLASH_SSN: track 60.9 -> 15.5 mm, vias 4 -> 2
- net +5V: track 45.7 -> 87.6 mm
- net ISP_MOSI: track 29.6 -> 69.7 mm, vias 2 -> 3
- net USER_FLASH_SCK: track 113.8 -> 80.0 mm, vias 2 -> 1
- net Net-(U8-~{DTR}): track 15.0 -> 47.7 mm, vias 2 -> 0
- net ardunio_d0: track 114.4 -> 85.4 mm
- net xclk: track 58.7 -> 84.9 mm, vias 1 -> 4
- net Net-(U5-vccd): track 38.6 -> 13.3 mm, vias 4 -> 1
- net +1V8: track 103.1 -> 79.2 mm, vias 2 -> 3
- net ISP_SSN: track 24.2 -> 47.4 mm, vias 0 -> 1
- net USER_SRAM_SSN: track 60.3 -> 81.7 mm
- net ardunio_d3: track 57.8 -> 78.7 mm, vias 2 -> 4
- net ardunio_a3: track 49.9 -> 30.3 mm, vias 2 -> 0
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Other:
- board text added: "5V"
- board text removed: "1.8V"
