File: KiCad_PCB/Riscduino_Debug_Rev1.1/Riscduino_Debug.kicad_sch (KiCad schematic)
At the start: 86 parts, among them J1 Conn_01x06_Pin, J10 USB_B_Micro, J11 Conn_01x10_Pin, J2 Conn_01x08_Pin, J3 Conn_01x01, J4 Conn_02x04_Odd_Even, J5 ISP, J6 Conn_01x01, J7 Conn_01x01, J8 Conn_01x01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

Commit message: Update
Parts:
- removed TP1: TestPoint, Connector_PinHeader_2.54mm:PinHeader_1x01_P2.54mm_Vertical, symbol Connector:TestPoint
- added R33: R, Resistor_SMD:R_0603_1608Metric_Pad0.98x0.95mm_HandSolder, symbol Device:R
Connections:
- net +1V8: no longer J2.5 (Pin_5)
- net +5V: now also J2.5 (Pin_5)
- net at C13.2: now also R33.1
Changed lines of the file:
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@@
     (stroke (width 0) (type default))
   )
+  (wire (pts (xy 200.152 284.48) (xy 203.2 284.48))
+    (stroke (width 0) (type default))
+  )
   (wire (pts (xy 44.196 252.73) (xy 49.784 252.73))
     (stroke (width 0) (type default))
@@
     (stroke (width 0) (type default))
   )
-  (wire (pts (xy 200.152 284.48) (xy 201.422 284.48))
-    (stroke (width 0) (type default))
-  )
   (wire (pts (xy 158.242 249.682) (xy 158.242 246.38))
     (stroke (width 0) (type default))
@@
     (stroke (width 0) (type default))
   )
+  (wire (pts (xy 210.82 284.48) (xy 218.694 284.48))
+    (stroke (width 0) (type default))
+  )
   (wire (pts (xy 178.562 257.81) (xy 178.562 259.08))
     (stroke (width 0) (type default))
@@
   )
   (text_box "Riscduino to ardunio Pin Mapping"
-    (at 290.83 302.26 0) (size 133.35 106.426)
+    (at 304.292 288.798 90) (size 106.426 133.35)
     (stroke (width 0) (type default))
     (fill (type none))
@@
     (effects (font (size 1.27 1.27)) (justify left bottom))
   )
+  (label "~{PS_RST}" (at 211.582 284.988 0) (fields_autoplaced)
+    (effects (font (size 1.27 1.27)) (justify left bottom))
+  )
+  (label "~{PS_RST}" (at 327.914 262.636 0) (fields_autoplaced)
+    (effects (font (size 1.27 1.27)) (justify left bottom))
+  )
   (label "+1.8VP" (at 72.898 252.73 0) (fields_autoplaced)
     (effects (font (size 1.27 1.27)) (justify left bottom))
@@
     )
   )
+  (symbol (lib_id "Device:R") (at 207.01 284.48 90) (unit 1)
+    (in_bom yes) (on_board yes) (dnp no) (fields_autoplaced)
+    (property "Reference" "R33" (at 207.01 280.162 90)
+      (effects (font (size 1.27 1.27)))
+    )
+    (property "Value" "R" (at 207.01 282.702 90)
+      (effects (font (size 1.27 1.27)))
+    )
+    (property "Footprint" "Resistor_SMD:R_0603_1608Metric_Pad0.98x0.95mm_HandSolder" (at 207.01 286.258 90)
+      (effects (font (size 1.27 1.27)) hide)
+    )
+    (property "Datasheet" "~" (at 207.01 284.48 0)
+      (effects (font (size 1.27 1.27)) hide)
+    )
+    (pin "1")
+    (pin "2")
+    (instances
+      (project "Riscduino_Debug"
+        (path "/3385a618-de98-459b-bc8d-0b8733b3fac9"
+          (reference "R33") (unit 1)
+        )
+      )
+    )
+  )
   (symbol (lib_id "Device:C") (at 80.01 210.566 0) (unit 1)
     (in_bom yes) (on_board yes) (dnp no)
@@
     )
   )
-  (symbol (lib_id "power:+1V8") (at 335.788 325.628 270) (unit 1)
-    (in_bom yes) (on_board yes) (dnp no) (fields_autoplaced)
-    (property "Reference" "#PWR059" (at 331.978 325.628 0)
-      (effects (font (size 1.27 1.27)) hide)
-    )
-    (property "Value" "+1.8V" (at 339.09 326.263 90)
-      (effects (font (size 1.27 1.27)) (justify left))
-    )
-    (property "Footprint" "" (at 335.788 325.628 0)
-      (effects (font (size 1.27 1.27)) hide)
-    )
-    (property "Datasheet" "" (at 335.788 325.628 0)
-      (effects (font (size 1.27 1.27)) hide)
-    )
-    (pin "1")
-    (instances
-      (project "Riscduino_Debug"
-        (path "/3385a618-de98-459b-bc8d-0b8733b3fac9"
-          (reference "#PWR059") (unit 1)
-        )
-      )
-    )
-  )
   (symbol (lib_id "power:GND") (at 158.242 259.842 0) (unit 1)
     (in_bom yes) (on_board yes) (dnp no) (fields_autoplaced)
@@
     )
   )
+  (symbol (lib_id "power:+5V") (at 335.788 325.628 270) (unit 1)
+    (in_bom yes) (on_board yes) (dnp no) (fields_autoplaced)
+    (property "Reference" "#PWR030" (at 331.978 325.628 0)
+      (effects (font (size 1.27 1.27)) hide)
+    )
+    (property "Value" "+5V" (at 339.598 326.263 90)
+      (effects (font (size 1.27 1.27)) (justify left))
+    )
+    (property "Footprint" "" (at 335.788 325.628 0)
+      (effects (font (size 1.27 1.27)) hide)
+    )
+    (property "Datasheet" "" (at 335.788 325.628 0)
+      (effects (font (size 1.27 1.27)) hide)
+    )
+    (pin "1")
+    (instances
+      (project "Riscduino_Debug"
+        (path "/3385a618-de98-459b-bc8d-0b8733b3fac9"
+          (reference "#PWR030") (unit 1)
+        )
+      )
+    )
+  )
   (symbol (lib_id "power:+3.3V") (at 347.726 99.822 0) (unit 1)
     (in_bom yes) (on_board yes) (dnp no) (fields_autoplaced)
@@
         )
       )
-    )
-  )
-  (symbol (lib_id "Connector:TestPoint") (at 201.422 284.48 270) (unit 1)
-    (in_bom yes) (on_board yes) (dnp no) (fields_autoplaced)
-    (property "Reference" "TP1" (at 206.502 283.21 90)
-      (effects (font (size 1.27 1.27)) (justify left))
-    )
-    (property "Value" "TestPoint" (at 206.502 285.75 90)
-      (effects (font (size 1.27 1.27)) (justify left))
-    )
-    (property "Footprint" "Connector_PinHeader_2.54mm:PinHeader_1x01_P2.54mm_Vertical" (at 201.422 289.56 0)
-      (effects (font (size 1.27 1.27)) hide)
-    )
-    (property "Datasheet" "~" (at 201.422 289.56 0)
-      (effects (font (size 1.27 1.27)) hide)
-    )
-    (pin "1")
-    (instances
-      (project "Riscduino_Debug"
-        (path "/3385a618-de98-459b-bc8d-0b8733b3fac9"
-          (reference "TP1") (unit 1)
-        )
-      )
