File: KiCad_PCB/Riscduino_Uno_Rev1.2/Riscduino_Uno.kicad_sch (KiCad schematic)
At the start: 95 parts, among them J1 Conn_01x06_Pin, J10 Conn_01x10_Pin, J11 USB_B_Micro, J2 Conn_01x08_Pin, J3 Conn_01x01, J4 Conn_02x04_Odd_Even, J5 ISP, J6 Conn_01x01, J7 Conn_01x01, J8 Conn_01x01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

Commit message: Rev Uno 1.2 update
Parts:
- removed H1, H2, H3, H4: MountingHole, MountingHole:MountingHole_3.2mm_M3, symbol Mechanical:MountingHole
- removed J1: Conn_01x06_Pin, Connector_PinHeader_2.54mm:PinHeader_1x06_P2.54mm_Vertical, symbol Connector:Conn_01x06_Pin
- removed J10: Conn_01x10_Pin, Connector_PinHeader_2.54mm:PinHeader_1x10_P2.54mm_Vertical, symbol Connector:Conn_01x10_Pin
- removed J2, J9: Conn_01x08_Pin, Connector_PinHeader_2.54mm:PinHeader_1x08_P2.54mm_Vertical, symbol Connector:Conn_01x08_Pin
- removed R1: 10K, Resistor_SMD:R_0603_1608Metric_Pad0.98x0.95mm_HandSolder, symbol Device:R
- removed R10, R17: 0E, Resistor_SMD:R_0603_1608Metric_Pad0.98x0.95mm_HandSolder, symbol Device:R
- removed R18: DNI, Resistor_SMD:R_0603_1608Metric_Pad0.98x0.95mm_HandSolder, symbol Device:R
- removed TP1: TestPoint, Connector_PinHeader_2.54mm:PinHeader_1x01_P2.54mm_Vertical, symbol Connector:TestPoint
- removed U1: MAX1232ESA+T, Package_SO:SOIC-8-1EP_3.9x4.9mm_P1.27mm_EP2.29x3mm, symbol MAX1232ESA+T:MAX1232ESA+T
- added J1: Conn_01x32_Pin, Riscduino.Library:Arduino_UNO_R3_WithMountingHoles, symbol Connector:Conn_01x32_Pin
- added J2: Conn_01x03_Pin, Connector_PinHeader_2.54mm:PinHeader_1x03_P2.54mm_Vertical, symbol Connector:Conn_01x03_Pin
- C3: value 0.1uf -> 10uF; footprint Capacitor_SMD:C_0603_1608Metric_Pad1.08x0.95mm_HandSolder -> Capacitor_SMD:C_0805_2012Metric_Pad1.18x1.45mm_HandSolder
- D1, D2, D3, D4, D5: footprint LED_SMD:LED_0805_2012Metric_Pad1.15x1.40mm_HandSolder -> Riscduino:LED_0805_2012Metric_Pad1.15x1.40mm_HandSolder
- D6: footprint LED_SMD:LED_0805_2012Metric_Pad1.15x1.40mm_HandSolder -> Riscduino.Library:LED_0805_2012Metric_Pad1.15x1.40mm_HandSolder
- RV1: footprint Potentiometer_THT:Potentiometer_Bourns_3296W_Vertical -> Riscduino.Library:Potentiometer_Bourns_3296W_Vertical
- X1: footprint Crystal:Crystal_SMD_Abracon_ABM8G-4Pin_3.2x2.5mm -> Riscduino:Crystal_SMD_Abracon_ABM8G-4Pin_3.2x2.5mm
Connections:
- net ~{PB_RST} is gone; now on net ~{RST}: R32.2, SW1.2
- net +3.3V: now also J1.4 (Pin_4); no longer C3.1
- net +5V: now also J1.5 (Pin_5), J2.2 (Pin_2); no longer C20.1, J11.1 (VBUS)
- net CARAVEL_FLASH_SCK: now also U5.25 (flash_clk); no longer U5.24 (flash_csb)
- net CARAVEL_FLASH_SSN: now also U5.24 (flash_csb); no longer U5.25 (flash_clk)
- net GND: now also J1.29 (Pin_29), J1.6 (Pin_6), J1.7 (Pin_7), J2.1 (Pin_1)
- net ardunio_a0: now also J1.9 (Pin_9)
- net ardunio_a1: now also J1.10 (Pin_10)
- net ardunio_a2: now also J1.11 (Pin_11)
- net ardunio_a3: now also J1.12 (Pin_12)
- net ardunio_a4: now also J1.13 (Pin_13), J1.31 (Pin_31)
- net ardunio_a5: now also J1.14 (Pin_14), J1.32 (Pin_32)
- net ardunio_d0: now also U8.2 (TXD), J1.15 (Pin_15)
- net ardunio_d1: now also U8.3 (RXD), J1.16 (Pin_16)
- net ardunio_d10: now also J1.25 (Pin_25)
- net ardunio_d11: now also J1.26 (Pin_26)
- net ardunio_d12: now also J1.27 (Pin_27)
- net ardunio_d13: now also J1.28 (Pin_28)
- net ardunio_d2: now also J1.17 (Pin_17)
- net ardunio_d3: now also J1.18 (Pin_18)
- net ardunio_d4: now also J1.19 (Pin_19)
- net ardunio_d5: now also J1.20 (Pin_20)
- net ardunio_d6: now also J1.21 (Pin_21)
- net ardunio_d7: now also J1.22 (Pin_22)
- net ardunio_d8: now also J1.23 (Pin_23)
- net ardunio_d9: now also J1.24 (Pin_24)
- net gpio: now also J1.1 (Pin_1)
- net mprj_io_12: now also J1.30 (Pin_30)
- net mprj_io_37: now also J1.8 (Pin_8)
- net xclk: now also J1.2 (Pin_2)
- net ~{RST}: now also C3.1, J1.3 (Pin_3)
- new net +5VP: C20.1, J11.1 (VBUS), J2.3 (Pin_3)
Other:
- note added: "USB or External 5V Selection USB Power - Short Pin-2 & Pin3 External Power: Connect 5V - Pin2 and Gnd - Pin1"
- moved on the sheet: J3, J6, J7, J8, R32

Commit message: Riscduino Uno Rev1.2
Parts:
- U2: footprint Package_SO:SOIC-8_5.23x5.23mm_P1.27mm -> Riscduino:SOIC-8_5.23x5.23mm_P1.27mm
- U4: footprint Package_SO:SOIC-8_5.23x5.23mm_P1.27mm -> Riscduino.Library:SOIC-8_5.23x5.23mm_P1.27mm
- U8: footprint Package_SO:SOIC-16_3.9x9.9mm_P1.27mm -> Riscduino:SOIC-16_3.9x9.9mm_P1.27mm
Connections:
- net gpio: no longer J1.1 (Pin_1)
- net mprj_io_11: now also J1.3 (Pin_3)
- net mprj_io_12: now also J1.2 (Pin_2)
- net mprj_io_5_ser_rx: now also J1.1 (Pin_1)
- net xclk: no longer J1.2 (Pin_2)
- net ~{RST}: no longer J1.3 (Pin_3)
Changed lines of the file:
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@@
     (stroke (width 0) (type default))
   )
-  (wire (pts (xy 316.484 321.818) (xy 323.85 321.818))
+  (wire (pts (xy 316.484 321.818) (xy 325.882 321.818))
     (stroke (width 0) (type default))
   )
@@
     (stroke (width 0) (type default))
   )
-  (wire (pts (xy 316.484 324.358) (xy 324.612 324.358))
+  (wire (pts (xy 316.484 324.358) (xy 325.882 324.358))
     (stroke (width 0) (type default))
   )
@@
     (stroke (width 0) (type default))
   )
-  (wire (pts (xy 316.484 319.278) (xy 323.85 319.278))
+  (wire (pts (xy 316.484 319.278) (xy 325.882 319.278))
     (stroke (width 0) (type default))
   )
@@
     )
   )
+  (global_label "mprj_io_5_ser_rx" (shape input) (at 325.882 319.278 0) (fields_autoplaced)
+    (effects (font (size 1.27 1.27)) (justify left))
+    (property "Intersheetrefs" "${INTERSHEET_REFS}" (at 344.572 319.278 0)
+      (effects (font (size 1.27 1.27)) (justify left) hide)
+    )
+  )
   (global_label "mprj_io_7" (shape input) (at 124.46 49.53 90) (fields_autoplaced)
     (effects (font (size 1.27 1.27)) (justify left))
@@
     )
   )
+  (global_label "mprj_io_12" (shape bidirectional) (at 325.882 321.818 0) (fields_autoplaced)
+    (effects (font (size 1.27 1.27)) (justify left))
+    (property "Intersheetrefs" "${INTERSHEET_REFS}" (at 340.2404 321.818 0)
+      (effects (font (size 1.27 1.27)) (justify left) hide)
+    )
+  )
   (global_label "mprj_io_26" (shape bidirectional) (at 384.81 354.33 0) (fields_autoplaced)
     (effects (font (size 1.27 1.27)) (justify left))
@@
     )
   )
-  (global_label "~{RST}" (shape bidirectional) (at 324.612 324.358 0) (fields_autoplaced)
-    (effects (font (size 1.27 1.27)) (justify left))
-    (property "Intersheetrefs" "${INTERSHEET_REFS}" (at 332.0762 324.358 0)
-      (effects (font (size 1.27 1.27)) (justify left) hide)
-    )
-  )
   (global_label "mprj_io_27" (shape bidirectional) (at 114.3 114.3 270) (fields_autoplaced)
     (effects (font (size 1.27 1.27)) (justify right))
@@
     )
   )
-  (global_label "gpio" (shape bidirectional) (at 323.85 319.278 0) (fields_autoplaced)
-    (effects (font (size 1.27 1.27)) (justify left))
-    (property "Intersheetrefs" "${INTERSHEET_REFS}" (at 331.9189 319.278 0)
-      (effects (font (size 1.27 1.27)) (justify left) hide)
-    )
-  )
   (global_label "mprj_io_14" (shape input) (at 80.01 60.96 180) (fields_autoplaced)
     (effects (font (size 1.27 1.27)) (justify right))
@@
     )
   )
-  (global_label "xclk" (shape bidirectional) (at 323.85 321.818 0) (fields_autoplaced)
-    (effects (font (size 1.27 1.27)) (justify left))
-    (property "Intersheetrefs" "${INTERSHEET_REFS}" (at 331.6771 321.818 0)
-      (effects (font (size 1.27 1.27)) (justify left) hide)
-    )
-  )
   (global_label "mprj_io_2_SDI" (shape input) (at 144.78 49.53 90) (fields_autoplaced)
     (effects (font (size 1.27 1.27)) (justify left))
@@
     )
   )
+  (global_label "mprj_io_11" (shape bidirectional) (at 325.882 324.358 0) (fields_autoplaced)
+    (effects (font (size 1.27 1.27)) (justify left))
+    (property "Intersheetrefs" "${INTERSHEET_REFS}" (at 340.2404 324.358 0)
+      (effects (font (size 1.27 1.27)) (justify left) hide)
+    )
+  )
   (symbol (lib_id "power:+3.3V") (at 346.964 169.164 0) (unit 1)
     (in_bom yes) (on_board yes) (dnp no) (fields_autoplaced)
@@
       (effects (font (size 1.27 1.27)) (justify left))
     )
-    (property "Footprint" "Package_SO:SOIC-16_3.9x9.9mm_P1.27mm" (at 182.372 290.83 0)
-      (effects (font (size 1.27 1.27)) (justify left) hide)
+    (property "Footprint" "Riscduino:SOIC-16_3.9x9.9mm_P1.27mm" (at 182.372 290.83 0)
+      (effects (font (size 1.27 1.27)) (justify left))
     )
     (property "Datasheet" "https://datasheet.lcsc.com/szlcsc/Jiangsu-Qin-Heng-CH340C_C84681.pdf" (at 172.212 256.54 0)
@@
       (effects (font (size 1.27 1.27)) (justify left))
     )
-    (property "Footprint" "Package_SO:SOIC-8_5.23x5.23mm_P1.27mm" (at 346.964 198.882 0)
+    (property "Footprint" "Riscduino.Library:SOIC-8_5.23x5.23mm_P1.27mm" (at 346.964 198.882 0)
       (effects (font (size 1.27 1.27)) hide)
     )
@@
       (effects (font (size 1.27 1.27)) (justify left))
     )
-    (property "Footprint" "Package_SO:SOIC-8_5.23x5.23mm_P1.27mm" (at 347.726 62.738 0)
+    (property "Footprint" "Riscduino:SOIC-8_5.23x5.23mm_P1.27mm" (at 347.726 62.738 0)
       (effects (font (size 1.27 1.27)) hide)
     )
