File: KiCad_PCB/Riscduino_Tester_Rev1.0/Riscduino_Tester.kicad_sch (KiCad schematic)
At the start: 90 parts, among them J1 ISP, J10 Conn_01x10_Pin, J11 Conn_01x03_Pin, J12 Conn_01x01, J13 Conn_02x16_Odd_Even, J14 Conn_02x16_Odd_Even, J2 Conn_01x06_Pin, J3 Conn_01x08_Pin, J4 Conn_01x01, J5 Conn_01x01, J6 Conn_02x04_Odd_Even, J7 Conn_01x01, J8 USB_B_Micro, J9 Conn_01x08_Pin, SW1 4Pin Round Button SPST Straig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, U1 W25Q32JVSS, U2 23LC1024-I/P, U4 LM1117MP-3.3, U5 CH340C, U6 LM1117S-ADJ, U7 W25Q32JVSS, X1 ASE-10.000MHZ-LC-T

Commit message: update
Parts:
- J13: renamed from J14; footprint Connector_PinHeader_2.54mm:PinHeader_2x16_P2.54mm_Vertical -> Riscduino:PinHeader_2x16_P2.54mm_Vertical_Swap
- J14: renamed from J13; footprint Connector_PinHeader_2.54mm:PinHeader_2x16_P2.54mm_Vertical -> Riscduino.Library:PinHeader_2x16_P2.54mm_Vertical_Swap
- renumbered C28 to C10, C36 to C11, C32 to C12, C12 to C13, C13 to C14, C34 to C15, C14 to C16, C20 to C18, C15 to C19, C30 to C2, C16 to C20, C18 to C21, C19 to C22, C21 to C23, C22 to C24, C33 to C3, C3 to C4, C2 to C5, C35 to C6, C4 to C7, C31 to C8, C29 to C9, D6 to D1, D4 to D3, D5 to D4, D3 to D5, D1 to D6, J2 to J1, J1 to J2, R34 to R1, R8 to R10, R26 to R15, R18 to R16, R24 to R17, R15 to R18, R27 to R19, R1 to R2, R17 to R20, R28 to R21, R25 to R22, R20 to R23, R21 to R24, R23 to R25, R22 to R26, R16 to R27, R19 to R28, R5 to R3, R2 to R5, R3 to R6, R32 to R7, R33 to R8, U4 to U3, U6 to U4, U7 to U6
