File: KiCad_PCB/Riscduino_Debug_Rev1.3/Riscduino_Debug_Rev1.3.kicad_pcb (KiCad board)
At the start: 2 copper layers, 76.7 x 53.6 mm, 93 parts, among them J1 Conn_01x06_Pin, J10 Conn_01x08_Pin, J11 Conn_01x10_Pin, J12 Conn_01x03_Pin, J13 Conn_01x01, J2 ISP, J3 Conn_01x08_Pin, J4 Conn_01x01, J5 Conn_01x01, J6 Conn_02x04_Odd_Even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

Commit message: Debug 1.3 BOM clean up
Parts:
- C1, C3, C4, C5, C8: value 0.1uf -> 0.1uF
- R11, R19, R20, R21: value 0 Ohm -> 0E
Changed lines of the file:
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@@
         (effects (font (size 1.016 1.016) (thickness 0.1524)))
     )
-    (fp_text value "0.1uf" (at 0 1.43 -90) (layer "F.Fab") hide
+    (fp_text value "0.1uF" (at 0 1.43 -90) (layer "F.Fab") hide
         (effects (font (size 1 1) (thickness 0.15)))
     )
@@
         (effects (font (size 1.016 1.016) (thickness 0.1524)))
     )
-    (fp_text value "0.1uf" (at 0 1.43 90) (layer "F.Fab") hide
+    (fp_text value "0.1uF" (at 0 1.43 90) (layer "F.Fab") hide
         (effects (font (size 1 1) (thickness 0.15)))
     )
@@
         (effects (font (size 1.016 1.016) (thickness 0.1524)))
     )
-    (fp_text value "0.1uf" (at 0 1.43 90) (layer "F.Fab") hide
+    (fp_text value "0.1uF" (at 0 1.43 90) (layer "F.Fab") hide
         (effects (font (size 1 1) (thickness 0.15)))
     )
@@
         (effects (font (size 1.016 1.016) (thickness 0.1524)))
     )
-    (fp_text value "0.1uf" (at 0 1.43 -270) (layer "F.Fab") hide
+    (fp_text value "0.1uF" (at 0 1.43 -270) (layer "F.Fab") hide
         (effects (font (size 1 1) (thickness 0.15)))
     )
@@
         (effects (font (size 1.016 1.016) (thickness 0.1524)))
     )
-    (fp_text value "0.1uf" (at 0 1.43 -180) (layer "F.Fab") hide
+    (fp_text value "0.1uF" (at 0 1.43 -180) (layer "F.Fab") hide
         (effects (font (size 1 1) (thickness 0.15)))
     )
@@
         (effects (font (size 1.016 1.016) (thickness 0.1524)) (justify mirror))
     )
-    (fp_text value "0 Ohm" (at 0 -1.43 90) (layer "B.Fab") hide
+    (fp_text value "0E" (at 0 -1.43 90) (layer "B.Fab") hide
         (effects (font (size 1 1) (thickness 0.15)) (justify mirror))
     )
@@
         (effects (font (size 1.016 1.016) (thickness 0.1524)) (justify mirror))
     )
-    (fp_text value "0 Ohm" (at -0.9652 5.4356) (layer "B.Fab") hide
+    (fp_text value "0E" (at -0.9652 5.4356) (layer "B.Fab") hide
         (effects (font (size 1 1) (thickness 0.15)) (justify mirror))
     )
@@
         (effects (font (size 1.016 1.016) (thickness 0.1524)) (justify mirror))
     )
-    (fp_text value "0 Ohm" (at 0 -1.43 90) (layer "B.Fab") hide
+    (fp_text value "0E" (at 0 -1.43 90) (layer "B.Fab") hide
         (effects (font (size 1 1) (thickness 0.15)) (justify mirror))
     )
@@
         (effects (font (size 1.016 1.016) (thickness 0.1524)) (justify mirror))
     )
-    (fp_text value "0 Ohm" (at 0 -1.43) (layer "B.Fab") hide
+    (fp_text value "0E" (at 0 -1.43) (layer "B.Fab") hide
         (effects (font (size 1 1) (thickness 0.15)) (justify mirror))
     )
