File: KiCad_PCB/Riscduino_Debug_Rev1.3/Riscduino_Debug_Rev1.3.kicad_sch (KiCad schematic)
At the start: 93 parts, among them J1 Conn_01x06_Pin, J10 Conn_01x08_Pin, J11 Conn_01x10_Pin, J12 Conn_01x03_Pin, J13 Conn_01x01, J2 ISP, J3 Conn_01x08_Pin, J4 Conn_01x01, J5 Conn_01x01, J6 Conn_02x04_Odd_Even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

Commit message: Debug 1.3 BOM clean up
Parts:
- C1, C3, C4, C5, C8: value 0.1uf -> 0.1uF
- R11, R19, R20, R21: value 0 Ohm -> 0E
Changed lines of the file:
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@@
   (symbol (lib_id "Device:C") (at 354.584 37.084 90) (unit 1)
     (in_bom yes) (on_board yes) (dnp no) (fields_autoplaced)
-    (property "Reference" "C8" (at 354.584 30.988 90)
+    (property "Reference" "C8" (at 354.584 30.48 90)
       (effects (font (size 1.27 1.27)))
     )
-    (property "Value" "0.1uf" (at 354.584 33.528 90)
+    (property "Value" "0.1uF" (at 354.584 33.02 90)
       (effects (font (size 1.27 1.27)))
     )
@@
       (effects (font (size 1.27 1.27)))
     )
-    (property "Value" "0 Ohm" (at 92.71 102.108 90)
+    (property "Value" "0E" (at 92.71 102.108 90)
       (effects (font (size 1.27 1.27)))
     )
@@
       (effects (font (size 1.27 1.27)))
     )
-    (property "Value" "0 Ohm" (at 179.832 128.27 90)
+    (property "Value" "0E" (at 179.832 128.27 90)
       (effects (font (size 1.27 1.27)))
     )
@@
       (effects (font (size 1.27 1.27)))
     )
-    (property "Value" "0.1uf" (at 353.822 169.672 90)
+    (property "Value" "0.1uF" (at 353.822 169.672 90)
       (effects (font (size 1.27 1.27)))
     )
@@
   (symbol (lib_id "Device:C") (at 80.518 311.912 90) (unit 1)
     (in_bom yes) (on_board yes) (dnp no) (fields_autoplaced)
-    (property "Reference" "C23" (at 80.518 305.562 90)
+    (property "Reference" "C23" (at 80.518 306.07 90)
       (effects (font (size 1.27 1.27)))
     )
-    (property "Value" "0.1uF" (at 80.518 308.102 90)
+    (property "Value" "0.1uF" (at 80.518 308.61 90)
       (effects (font (size 1.27 1.27)))
     )
@@
       (effects (font (size 1.27 1.27)))
     )
-    (property "Value" "0 Ohm" (at 207.518 282.702 90)
+    (property "Value" "0E" (at 207.518 282.702 90)
       (effects (font (size 1.27 1.27)))
     )
@@
       (effects (font (size 1.27 1.27)) (justify left))
     )
-    (property "Value" "0.1uf" (at 501.65 71.247 0)
+    (property "Value" "0.1uF" (at 501.65 71.247 0)
       (effects (font (size 1.27 1.27)) (justify left))
     )
@@
       (effects (font (size 1.27 1.27)))
     )
-    (property "Value" "0 Ohm" (at 98.044 141.224 90)
+    (property "Value" "0E" (at 98.044 141.224 90)
       (effects (font (size 1.27 1.27)))
     )
@@
   (symbol (lib_id "Device:C") (at 369.57 252.73 0) (unit 1)
     (in_bom yes) (on_board yes) (dnp no) (fields_autoplaced)
-    (property "Reference" "C3" (at 373.38 251.46 0)
+    (property "Reference" "C3" (at 373.38 252.095 0)
       (effects (font (size 1.27 1.27)) (justify left))
     )
-    (property "Value" "0.1uf" (at 373.38 254 0)
+    (property "Value" "0.1uF" (at 373.38 254.635 0)
       (effects (font (size 1.27 1.27)) (justify left))
     )
@@
       (effects (font (size 1.27 1.27)))
     )
-    (property "Value" "0.1uf" (at 354.584 100.33 90)
+    (property "Value" "0.1uF" (at 354.584 100.33 90)
       (effects (font (size 1.27 1.27)))
     )
