File: KiCad_PCB/Riscduino_Debug_Rev1.4/Riscduino_Debug_Rev1.4.kicad_sch (KiCad schematic)
At the start: 96 parts, among them J1 Conn_01x06_Pin, J10 Conn_01x08_Pin, J11 Conn_01x10_Pin, J12 Conn_01x03_Pin, J13 Conn_01x01, J2 ISP, J3 Conn_01x08_Pin, J4 Conn_01x01, J5 Conn_01x01, J6 Conn_02x04_Odd_Even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

Commit message: update
Parts:
- removed R36, R37: 10K, Riscduino.Library:R_0603_1608Metric_Pad0.98x0.95mm_HandSolder, symbol Device:R
- removed U9: LSM6DSL, Package_LGA:LGA-14_3x2.5mm_P0.5mm_LayoutBorder3x4y, symbol Sensor_Motion:LSM6DSL
- added J14: Conn_01x06_Male_Header, Riscduino.Library:PinHeader_1x06_P2.54mm_Vertical, symbol Connector:Conn_01x06_Pin
- added J15: Conn_01x10_Male_Header, Riscduino.Library:PinHeader_1x10_P2.54mm_Vertical, symbol Connector:Conn_01x10_Pin
- added J16, J17: Conn_01x08_Male_Header, Riscduino.Library:PinHeader_1x08_P2.54mm_Vertical, symbol Connector:Conn_01x08_Pin
- J1: value Conn_01x06_Pin -> Conn_01x06_Female_Header
- J10, J3: value Conn_01x08_Pin -> Conn_01x08_Female_Header
- J11: value Conn_01x10_Pin -> Conn_01x10_Female_Header
Connections:
- net +3.3V: now also J16.4 (Pin_4)
- net +5V: now also J16.5 (Pin_5)
- net GND: now also J15.7 (Pin_7), J16.6 (Pin_6), J16.7 (Pin_7)
- net ardunio_a0: now also J14.1 (Pin_1)
- net ardunio_a1: now also J14.2 (Pin_2)
- net ardunio_a2: now also J14.3 (Pin_3)
- net ardunio_a3: now also J14.4 (Pin_4)
- net ardunio_a4: now also J14.5 (Pin_5), J15.9 (Pin_9)
- net ardunio_a5: now also J14.6 (Pin_6), J15.10 (Pin_10)
- net ardunio_d0: now also J17.1 (Pin_1)
- net ardunio_d1: now also J17.2 (Pin_2)
- net ardunio_d10: now also J15.3 (Pin_3)
- net ardunio_d11: now also J15.4 (Pin_4)
- net ardunio_d12: now also J15.5 (Pin_5)
- net ardunio_d13: now also J15.6 (Pin_6)
- net ardunio_d2: now also J17.3 (Pin_3)
- net ardunio_d3: now also J17.4 (Pin_4)
- net ardunio_d4: now also J17.5 (Pin_5)
- net ardunio_d5: now also J17.6 (Pin_6)
- net ardunio_d6: now also J17.7 (Pin_7)
- net ardunio_d7: now also J17.8 (Pin_8)
- net ardunio_d8: now also J15.1 (Pin_1)
- net ardunio_d9: now also J15.2 (Pin_2)
- net mprj_io_11: now also J16.3 (Pin_3)
- net mprj_io_12: now also J16.2 (Pin_2)
- net mprj_io_30: now also J15.8 (Pin_8)
- net mprj_io_37: now also J16.8 (Pin_8)
- net mprj_io_5_ser_rx: now also J16.1 (Pin_1)
Other:
- moved on the sheet: H1, J1, J10, J11, J3
