File: KiCad_PCB/Riscduino_Fpga_Rev1.1/Riscduino_Fpga_Rev1.1.kicad_sch (KiCad schematic)
At the start: 103 parts, among them J1 Conn_01x06_Female_Header, J10 Conn_01x08_Female_Header, J11 Conn_01x10_Female_Header, J12 Conn_01x03_Male_Header, J13 Conn_01x01, J14 Conn_01x06_Male_Header, J15 Conn_01x10_Male_Header, J16 Conn_01x08_Male_Header, J17 Conn_01x08_Male_Header, J18 Conn_02x15_Male_Header, J19 Micro_SD_Card, J2 Conn_01x03_Male_Header, J20 USB Type A Female, J21 USB_B_Micro_Female, J22 Conn_02x06_Odd_Even, J3 Conn_01x08_Female_Header, J4 Conn_01x01, J5 Conn_02x15_Male_Header, J6 Conn_02x04_Male_Header, J7 Conn_01x08_Female_Header, J8 Conn_01x01, J9 USB_B_Micro_Female, SW1 4Pin Round Button SPST Straig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, SW2 SW_DIP_x04, SW3 4Pin Round Button SPST Straig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, SW4 4Pin Round Button SPST Straig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, SW5 4Pin Round Button SPST Straig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, SW6 4Pin Round Button SPST Straig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, SW7 4Pin Round Button SPST Straig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, SW8 4Pin Round Button SPST Straig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, U1 APX811-29UG-7, U3 23LC1024-I/P, U5 CH340C, U6 LM1117MP-3.3, U8 W25Q32JVSS, X1 ASE-10.000MHZ-LC-T

Commit message: Update
Parts:
- J22: value Conn_02x06_Odd_Even -> Conn_02x06_Male_Header
Changed lines of the file:
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@@
       (effects (font (size 1.27 1.27)))
     )
-    (property "Value" "Conn_02x06_Odd_Even" (at 373.38 89.408 0)
+    (property "Value" "Conn_02x06_Male_Header" (at 373.38 89.408 0)
       (effects (font (size 1.27 1.27)))
     )
